Commit message: 修改里程計買轉一圈幾個訊號參數，地圖在掃到小於多少距離忽略

File: src/example_2/description/ros2_control/diffbot.ros2_control.xacro (robot description, xacro)
@@ -12,5 +12,5 @@
           <param name="baud_rate">115200</param>
           <param name="timeout_ms">1000</param>
-          <param name="enc_counts_per_rev">880</param>
+          <param name="enc_counts_per_rev">220</param>
           <!-- <param name="example_param_hw_start_duration_sec">0</param>
           <param name="example_param_hw_stop_duration_sec">3.0</param> -->

File: src/ros2_control_demo_description/diffbot/urdf/mydiffbot_description.urdf.xacro (robot description, xacro)
@@ -166,5 +166,5 @@
         <cylinder length="0.03" radius="0.03"/>
       </geometry>
-      <material name="gray"/>
+      <material name="black"/>
     </visual>
     <collision>

Commit message: 改一些里程計的部份，和tf左右輪錯誤修該

File: src/example_2/description/ros2_control/diffbot.ros2_control.xacro (robot description, xacro)
@@ -9,6 +9,7 @@
           <param name="right_wheel_name">right_wheel_joint</param>
           <param name="loop_rate">30.0</param>
-          <param name="device">/dev/ttyUSB0</param>
-          <param name="baud_rate">115200</param>
+          <!-- <param name="device">/dev/ttyUSB0</param> -->
+          <param name="device">/dev/serial/by-path/platform-xhci-hcd.0-usb-0:1:1.0-port0</param>
+	  <param name="baud_rate">115200</param>
           <param name="timeout_ms">1000</param>
           <param name="enc_counts_per_rev">220</param>

File: src/ros2_control_demo_description/diffbot/urdf/mydiffbot_description.urdf.xacro (robot description, xacro)
@@ -45,5 +45,5 @@
       <child link="${prefix}left_wheel"/>
       <!-- <origin xyz="0 -${base_width/2} ${z_offset}" rpy="0 0 0"/> -->
-      <origin xyz="0.055 ${(-base_width/2)-(wheel_len/2)-0.001} 0" rpy="0 0 0"/>
+      <origin xyz="0.055 ${(base_width/2)+(wheel_len/2)-0.001} 0" rpy="0 0 0"/>
       <axis xyz="0 1 0"/>
       <dynamics damping="0.2"/>
@@ -75,5 +75,5 @@
       <child link="${prefix}right_wheel"/>
       <!-- <origin xyz="0 ${base_width/2} ${z_offset}" rpy="0 0 0"/> -->
-      <origin xyz="0.055 ${(base_width/2)+(wheel_len/2)+0.001} 0" rpy="0 0 0"/>
+      <origin xyz="0.055 ${(-base_width/2)-(wheel_len/2)+0.001} 0" rpy="0 0 0"/>
       <axis xyz="0 1 0"/>
       <dynamics damping="0.2"/>

Commit message: 模擬可以鍵盤遙控車子

File: src/example_2/description/ros2_control/diffbot.ros2_control.xacro (robot description, xacro)
@@ -2,37 +2,44 @@
 <robot xmlns:xacro="http://www.ros.org/wiki/xacro">
   <xacro:macro name="diffbot_ros2_control" params="name prefix use_mock_hardware">
-    <ros2_control name="${name}" type="system">
-      <xacro:unless value="${use_mock_hardware}">
-        <hardware>
-          <plugin>ros2_control_demo_example_2/DiffBotSystemHardware</plugin>
-          <param name="left_wheel_name">left_wheel_joint</param>
-          <param name="right_wheel_name">right_wheel_joint</param>
-          <param name="loop_rate">30.0</param>
-          <!-- <param name="device">/dev/ttyUSB0</param> -->
-          <param name="device">/dev/serial/by-path/platform-xhci-hcd.0-usb-0:1:1.0-port0</param>
-	  <param name="baud_rate">115200</param>
-          <param name="timeout_ms">1000</param>
-          <param name="enc_counts_per_rev">220</param>
-          <!-- <param name="example_param_hw_start_duration_sec">0</param>
-          <param name="example_param_hw_stop_duration_sec">3.0</param> -->
-        </hardware>
-      </xacro:unless>
-      <xacro:if value="${use_mock_hardware}">
-        <hardware>
-          <plugin>mock_components/GenericSystem</plugin>
-          <param name="calculate_dynamics">true</param>
-        </hardware>
-      </xacro:if>
-      <joint name="${prefix}left_wheel_joint">
-        <command_interface name="velocity"/>
-        <state_interface name="position"/>
-        <state_interface name="velocity"/>
-      </joint>
-      <joint name="${prefix}right_wheel_joint">
-        <command_interface name="velocity"/>
-        <state_interface name="position"/>
-        <state_interface name="velocity"/>
-      </joint>
-    </ros2_control>
+      <ros2_control name="${name}" type="system">
+        <xacro:unless value="${use_mock_hardware}">
+          <hardware>
+            <plugin>ros2_control_demo_example_2/DiffBotSystemHardware</plugin>
+            <param name="left_wheel_name">left_wheel_joint</param>
+            <param name="right_wheel_name">right_wheel_joint</param>
+            <param name="loop_rate">30.0</param>
+            <!-- <param name="device">/dev/ttyUSB0</param> -->
+            <param name="device">/dev/serial/by-path/platform-xhci-hcd.0-usb-0:1:1.0-port0</param>
+            <param name="baud_rate">115200</param>
+            <param name="timeout_ms">1000</param>
+            <param name="enc_counts_per_rev">220</param>
+            <!-- <param name="example_param_hw_start_duration_sec">0</param>
+            <param name="example_param_hw_stop_duration_sec">3.0</param> -->
+          </hardware>
+        </xacro:unless>
+        <xacro:if value="${use_mock_hardware}">
+          <hardware>
+            <!-- <plugin>mock_components/GenericSystem</plugin> -->
+            <plugin>gz_ros2_control/GazeboSimSystem</plugin>
+            <param name="calculate_dynamics">true</param>
+          </hardware>
+        </xacro:if>
+        <joint name="${prefix}left_wheel_joint">
+          <command_interface name="velocity"/>
+          <state_interface name="position"/>
+          <state_interface name="velocity"/>
+        </joint>
+        <joint name="${prefix}right_wheel_joint">
+          <command_interface name="velocity"/>
+          <state_interface name="position"/>
+          <state_interface name="velocity"/>
+        </joint>
+      </ros2_control>
+    <gazebo>
+      <plugin name="gz_ros2_control::GazeboSimROS2ControlPlugin" filename="libgz_ros2_control-system.so">
+        <parameters>$(find ros2_control_demo_example_2)/config/diffbot_controllers.yaml</parameters>
+        <!-- <parameters>$(find ros2_control_demo_example_2)/config/gaz_ros2_ctl_use_sim.yaml</parameters> -->
+      </plugin>
+    </gazebo>
   </xacro:macro>
 </robot>

File: src/example_2/description/urdf/diffbot.urdf.xacro (robot description, xacro)
@@ -4,4 +4,5 @@
   <xacro:arg name="prefix" default="" />
   <xacro:arg name="use_mock_hardware" default="false" />
+  <xacro:arg name="sim_mode" default="false" />
   <xacro:include filename="$(find ros2_control_demo_description)/diffbot/urdf/mydiffbot_description.urdf.xacro" />
   <!-- Import Rviz colors -->
