Commit message: 增加激光雷達功能

File: src/ros2_control_demo_description/diffbot/urdf/mydiffbot_description.urdf.xacro (robot description, xacro)
@@ -155,4 +155,29 @@
       </inertial>
     </link>
+  <joint name="${prefix}laser_joint" type="fixed">
+    <parent link="${prefix}base_link"/>
+    <child  link="${prefix}laser"/>
+    <origin xyz="0.059 0 0.1025" rpy="0 0 0"/>
+  </joint>
+  <link name="${prefix}laser">
+    <visual>
+      <origin xyz="0 0 0" rpy="0 0 0"/>
+      <geometry>
+        <cylinder length="0.03" radius="0.03"/>
+      </geometry>
+      <material name="gray"/>
+    </visual>
+    <collision>
+      <origin xyz="0 0 0" rpy="0 0 0"/>
+      <geometry>
+        <cylinder length="0.03" radius="0.03"/>
+      </geometry>
+    </collision>
+    <inertial>
+      <origin xyz="0 0 0" rpy="0 0 0"/>
+      <mass value="0.2"/>
+      <inertia ixx="0.0001" ixy="0.0" ixz="0.0" iyy="0.0001" iyz="0.0" izz="0.0001"/>
+    </inertial>
+  </link>
   </xacro:macro>
 </robot>

Commit message: 翻轉激光雷達方向

File: src/ros2_control_demo_description/diffbot/urdf/mydiffbot_description.urdf.xacro (robot description, xacro)
@@ -158,5 +158,5 @@
     <parent link="${prefix}base_link"/>
     <child  link="${prefix}laser"/>
-    <origin xyz="0.059 0 0.1025" rpy="0 0 0"/>
+    <origin xyz="0.059 0 0.1025" rpy="0 0 3.1415926"/>
   </joint>
   <link name="${prefix}laser">

Commit message: urdf修改位置

File: src/ros2_control_demo_description/diffbot/urdf/mydiffbot_description.urdf.xacro (robot description, xacro)
@@ -22,4 +22,11 @@
     <!-- Base Link -->
     <link name="${prefix}base_link">
+    </link>
+    <joint name="${prefix}chassis_joint" type="fixed">
+      <parent link="${prefix}base_link"/>
+      <child link="${prefix}chassis"/>
+      <origin xyz="0 0 ${wheel_radius}" rpy="0 0 0"/>
+    </joint>
+    <link name="${prefix}chassis">
       <collision>
         <origin xyz="0 0 0" rpy="0 0 0"/>
@@ -45,5 +52,5 @@
       <child link="${prefix}left_wheel"/>
       <!-- <origin xyz="0 -${base_width/2} ${z_offset}" rpy="0 0 0"/> -->
-      <origin xyz="0.055 ${(base_width/2)+(wheel_len/2)-0.001} 0" rpy="0 0 0"/>
+      <origin xyz="0.055 ${(base_width/2)+(wheel_len/2)-0.001} ${wheel_radius}" rpy="0 0 0"/>
       <axis xyz="0 1 0"/>
       <dynamics damping="0.2"/>
@@ -75,5 +82,5 @@
       <child link="${prefix}right_wheel"/>
       <!-- <origin xyz="0 ${base_width/2} ${z_offset}" rpy="0 0 0"/> -->
-      <origin xyz="0.055 ${(-base_width/2)-(wheel_len/2)+0.001} 0" rpy="0 0 0"/>
+      <origin xyz="0.055 ${(-base_width/2)-(wheel_len/2)+0.001} ${wheel_radius}" rpy="0 0 0"/>
       <axis xyz="0 1 0"/>
       <dynamics damping="0.2"/>
@@ -105,5 +112,6 @@
       <child link="${prefix}caster_right_wheel"/>
       <!-- <origin xyz="${base_width/2 - caster_wheel_radius} 0 ${z_offset}" rpy="0 0 0"/> -->
-      <origin xyz="-0.05 0.05 -${wheel_radius-0.0075}" rpy="0 0 0"/>
+      <!-- <origin xyz="-0.05 0.05 -${wheel_radius-0.0075}" rpy="0 0 0"/> -->
+      <origin xyz="-0.05 0.05 ${caster_wheel_radius}" rpy="0 0 0"/>
     </joint>
     <!-- caster right wheel Link -->
@@ -132,5 +140,6 @@
       <child link="${prefix}caster_left_wheel"/>
       <!-- <origin xyz="${-base_width/2 + caster_wheel_radius} 0 ${z_offset}" rpy="0 0 0"/> -->
-      <origin xyz="-0.05 -0.05 -${wheel_radius-0.0075}" rpy="0 0 0"/>
+      <!-- <origin xyz="-0.05 -0.05 -${wheel_radius-0.0075}" rpy="0 0 0"/> -->
+      <origin xyz="-0.05 -0.05 ${caster_wheel_radius}" rpy="0 0 0"/>
     </joint>
     <!-- caster left wheel Link -->
@@ -158,5 +167,5 @@
     <parent link="${prefix}base_link"/>
     <child  link="${prefix}laser"/>
-    <origin xyz="0.059 0 0.1025" rpy="0 0 3.1415926"/>
+    <origin xyz="0.059 0 0.136" rpy="0 0 0"/> <!--z 0.1025+0.335(輪胎半徑)-->
   </joint>
   <link name="${prefix}laser">

Commit message: 重要：修改ros2_control.yaml 左右輪之間的距離、模型有稍微調整

File: src/ros2_control_demo_description/diffbot/urdf/mydiffbot_description.urdf.xacro (robot description, xacro)
@@ -10,5 +10,5 @@
     <xacro:property name="base_width" value="0.15" />
     <xacro:property name="base_length" value="0.18" />
-    <xacro:property name="base_height" value="0.07135" />
+    <xacro:property name="base_height" value="0.067" />
     <xacro:property name="wheel_mass" value="0.3" />
     <!-- arbitrary value for wheel mass -->
@@ -165,7 +165,7 @@
     </link>
   <joint name="${prefix}laser_joint" type="fixed">
-    <parent link="${prefix}base_link"/>
+    <parent link="${prefix}chassis"/>
     <child  link="${prefix}laser"/>
-    <origin xyz="0.059 0 0.136" rpy="0 0 0"/> <!--z 0.1025+0.335(輪胎半徑)-->
+    <origin xyz="0.050 -0.0105 0.12" rpy="0 0 3.1415926"/> <!--z 0.1025+0.335(輪胎半徑)-->
   </joint>
   <link name="${prefix}laser">
@@ -173,5 +173,5 @@
       <origin xyz="0 0 0" rpy="0 0 0"/>
       <geometry>
-        <cylinder length="0.03" radius="0.03"/>
+        <cylinder length="0.024" radius="0.0345"/>
       </geometry>
       <material name="black"/>
@@ -180,5 +180,5 @@
       <origin xyz="0 0 0" rpy="0 0 0"/>
       <geometry>
-        <cylinder length="0.03" radius="0.03"/>
+        <cylinder length="0.024" radius="0.0345"/>
       </geometry>
     </collision>

Commit message: 建圖問題修改好了（模型錯誤導致激光雷達偵測到的牆壁隨著車子旋轉而旋轉）,基本導航也可以（但是要避障的版本還沒有）

File: src/ros2_control_demo_description/diffbot/urdf/mydiffbot_description.urdf.xacro (robot description, xacro)
@@ -10,8 +10,8 @@
     <xacro:property name="base_width" value="0.15" />
     <xacro:property name="base_length" value="0.18" />
-    <xacro:property name="base_height" value="0.067" />
+    <xacro:property name="base_height" value="0.07135" />
     <xacro:property name="wheel_mass" value="0.3" />
     <!-- arbitrary value for wheel mass -->
-    <xacro:property name="wheel_len" value="0.020" />
+    <xacro:property name="wheel_len" value="0.025" />
     <xacro:property name="wheel_radius" value="0.0335" />
     <xacro:property name="caster_wheel_mass" value="0.1" />
@@ -30,5 +30,5 @@
     <link name="${prefix}chassis">
       <collision>
-        <origin xyz="0 0 0" rpy="0 0 0"/>
+        <origin xyz="0 0 ${base_height/2}" rpy="0 0 0"/>
         <geometry>
           <box size="${base_length} ${base_width} ${base_height}"/>
@@ -52,5 +52,5 @@
       <child link="${prefix}left_wheel"/>
       <!-- <origin xyz="0 -${base_width/2} ${z_offset}" rpy="0 0 0"/> -->
-      <origin xyz="0.055 ${(base_width/2)+(wheel_len/2)-0.001} ${wheel_radius}" rpy="0 0 0"/>
+      <origin xyz="0.055 ${(base_width/2)+(wheel_len/2)+0.003} ${wheel_radius}" rpy="0 0 0"/>
       <axis xyz="0 1 0"/>
       <dynamics damping="0.2"/>
@@ -82,5 +82,5 @@
       <child link="${prefix}right_wheel"/>
       <!-- <origin xyz="0 ${base_width/2} ${z_offset}" rpy="0 0 0"/> -->
-      <origin xyz="0.055 ${(-base_width/2)-(wheel_len/2)+0.001} ${wheel_radius}" rpy="0 0 0"/>
+      <origin xyz="0.055 ${(-base_width/2)-(wheel_len/2)-0.003} ${wheel_radius}" rpy="0 0 0"/>
       <axis xyz="0 1 0"/>
       <dynamics damping="0.2"/>
@@ -164,8 +164,9 @@
       </inertial>
     </link>
+  <!-- laser -->
   <joint name="${prefix}laser_joint" type="fixed">
     <parent link="${prefix}chassis"/>
     <child  link="${prefix}laser"/>
-    <origin xyz="0.050 -0.0105 0.12" rpy="0 0 3.1415926"/> <!--z 0.1025+0.335(輪胎半徑)-->
+    <origin xyz="0.055 0 0.12" rpy="0 0 3.1415926"/> <!--z 0.1025+0.335(輪胎半徑)-->
   </joint>
   <link name="${prefix}laser">

Commit message: 模擬功能完成 可以導航建圖

File: src/ros2_control_demo_description/diffbot/urdf/mydiffbot_description.urdf.xacro (robot description, xacro)
@@ -55,5 +55,5 @@
       <axis xyz="0 1 0"/>
       <dynamics damping="0.2"/>
-      <limit effort="100" velocity="1.0"/>
+      <limit effort="100" velocity="10.0"/>
     </joint>
     <!-- left wheel Link -->
@@ -85,5 +85,5 @@
       <axis xyz="0 1 0"/>
       <dynamics damping="0.2"/>
-      <limit effort="100" velocity="1.0"/>
+      <limit effort="100" velocity="10.0"/>
     </joint>
     <!-- right wheel Link -->
@@ -190,4 +190,27 @@
     </inertial>
   </link>
+  <!-- gz lidar -->
+  <gazebo reference="${prefix}laser">
+    <sensor name="laser" type="gpu_lidar">
+      <pose> 0 0 0 0 0 0 </pose>
+      <visualize>false</visualize>
+      <update_rate>10</update_rate>
+      <topic>scan</topic>
+      <gz_frame_id>laser</gz_frame_id>
+      <lidar>
+        <scan>
+          <horizontal>
+            <samples>360</samples>
+            <min_angle>-${PI}</min_angle>
+            <max_angle>${PI}</max_angle>
+          </horizontal>
+        </scan>
+        <range>
+          <min>0.5</min>
+          <max>12.0</max>
+        </range>
+      </lidar>
+    </sensor>
+  </gazebo>
   </xacro:macro>
 </robot>
